File: micromouse.kicad_pcb (KiCad board)
At the start: 2 copper layers, 11 parts, among them SW1 SW_SPST, SW2 SW_Push, U1 BUCK, U2 STM32 Blackpill, U3 N20 encoder right, U4 N20 encoder left, U5 TB6612FNG, U6 VL53L0X left, U7 VL53L0X right, U8 VL53L0X middle

Commit message: schematic and footprint changes
Parts:
- removed SW1: SW_SPST, SPST:JUDCOSPST
- added J1: XT60-M, XT60:AMASS_XT60-M, F.Cu at (205.7, 131.0)
- added REF**: MountingHole_3.2mm_M3_Pad_TopBottom, MountingHole:MountingHole_3.2mm_M3_Pad_TopBottom, F.Cu at (115.1, 58.4)
- added REF**: MountingHole_3.2mm_M3_Pad_TopBottom, MountingHole:MountingHole_3.2mm_M3_Pad_TopBottom, F.Cu at (115.1, 150.4)
- added REF**: MountingHole_3.2mm_M3_Pad_TopBottom, MountingHole:MountingHole_3.2mm_M3_Pad_TopBottom, F.Cu at (206.8, 58.4)
- added REF**: MountingHole_3.2mm_M3_Pad_TopBottom, MountingHole:MountingHole_3.2mm_M3_Pad_TopBottom, F.Cu at (206.8, 150.4)
- U3, U4: footprint Connector_PinHeader_2.00mm:PinHeader_1x06_P2.00mm_Vertical -> Connector_PinHeader_2.54mm:PinHeader_1x06_P2.54mm_Vertical
- moved U7 182.3 mm to (200.4, 69.1), turned to -90 degrees
- moved U8 143.1 mm to (152.0, 64.8)
- moved U2 131.0 mm to (187.5, 93.7), turned to 180 degrees
- moved SW2 112.6 mm to (184.8, 79.5), turned to 90 degrees
- moved U6 98.6 mm to (121.4, 86.9), turned to 90 degrees
- moved U3 86.3 mm to (208.5, 99.4)
- moved U4 84.0 mm to (113.3, 99.4)
- moved U1 64.3 mm to (162.9, 133.9), turned to 180 degrees
- moved U5 63.1 mm to (140.7, 130.9), turned to 90 degrees
- moved ACC1 36.1 mm to (171.9, 87.0), turned to 90 degrees
Other:
- board outline added: 100 x 100 mm

Commit message: routing
Connections:
- U5 pad 4: AO1  -> AO1
Routing:
- net GND: track 0.00 -> 324.6 mm, vias 0 -> 4
- net 3.3v: track 0.00 -> 222.4 mm
- net SDA: track 0.00 -> 161.2 mm
- net SCL: track 0.00 -> 126.4 mm
- net AO1: track 0.00 -> 85.5 mm
- net STBY: track 0.00 -> 79.5 mm, vias 0 -> 1
- net AO2: track 0.00 -> 77.0 mm
- net 7.4v: track 0.00 -> 77.0 mm
- net BO1: track 0.00 -> 75.6 mm
- net XSHUT 3: track 0.00 -> 69.7 mm
- net encoder A1: track 0.00 -> 69.1 mm, vias 0 -> 1
- net 5v: track 0.00 -> 65.8 mm
- net encoder B1: track 0.00 -> 57.1 mm, vias 0 -> 1
- net encoder B2: track 0.00 -> 46.3 mm
- net BO2: track 0.00 -> 42.0 mm
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
Commit message: ll
Parts:
- added SW3: SW_Push, push button:push_button, F.Cu at (136.9, 78.5)
- U5: footprint TB6612FNG:TB6612FNG -> Tb6612fng:TB6612FNG
- moved U3 13.5 mm to (195.1, 99.8)
- moved U4 12.7 mm to (126.0, 99.8)
Connections:
- U2 pad 13: unconnected-(U2-B5-Pad13) -> push button 1
Routing:
- net AO1: track 85.5 -> 0.00 mm
- net AO2: track 77.0 -> 0.00 mm
- net GND: track 324.6 -> 253.6 mm, vias 4 -> 1
- net encoder B1: track 57.1 -> 0.60 mm, vias 1 -> 0
- net 3.3v: track 222.4 -> 183.8 mm
- net push button 1: track 0.00 -> 30.5 mm
- net SDA: track 161.2 -> 130.9 mm, vias 0 -> 2
- net encoder B2: track 46.3 -> 25.3 mm
- net STBY: track 79.5 -> 60.9 mm, vias 1 -> 0
- net encoder A1: track 69.1 -> 52.7 mm
- net encoder A2: track 33.7 -> 21.7 mm, vias 1 -> 0
- net XSHUT 3: track 69.7 -> 79.8 mm
- net BO2: track 42.0 -> 37.4 mm, vias 0 -> 1
- net BO1: track 75.6 -> 80.1 mm
Other:
- outline, holes or cut-outs redrawn
- board text added: "3.3v"
- board text added: "5V"
- board text added: "5v"
- board text added: "A0"
- board text added: "A1"
- board text added: "A10"
- board text added: "A11"
- board text added: "A12"
- board text added: "A15"
- board text added: "A2"
- board text added: "A3"
- board text added: "A4"
- board text added: "A5"
- board text added: "A6"
- board text added: "A7"
- board text added: "A8"
- board text added: "A9"
- board text added: "B0"
- board text added: "B1"
- board text added: "B10"
- board text added: "B13"
- board text added: "B14"
- board text added: "B15"
- board text added: "B2"
- board text added: "B3"
- board text added: "B4"
- board text added: "B5"
- board text added: "B6"
- board text added: "B7"
- board text added: "B8"
- board text added: "B9"
- board text added: "C13"
- board text added: "C14"
- board text added: "C15"
- board text added: "GND"
- board text added: "R"
- board text added: "STBY"
- board text added: "VB"

Commit message: pcb changes
Parts:
- removed REF** (x4): MountingHole_3.2mm_M3_Pad_TopBottom, MountingHole:MountingHole_3.2mm_M3_Pad_TopBottom
- added SW4: SW_SPDT_312, slide switch:SLIDE SW, F.Cu at (188.2, 65.1)
- U5: footprint Tb6612fng:TB6612FNG -> TB6612FNG:TB6612FNG
- moved U2 52.3 mm to (171.6, 143.5), turned to 90 degrees
- moved U1 20.0 mm to (182.6, 131.1)
- moved U5 12.9 mm to (132.3, 140.7), turned to 180 degrees
- moved U4 10.2 mm to (136.1, 99.8)
- moved U3 9.40 mm to (185.7, 99.8)
- moved SW2 3.57 mm to (185.0, 83.1)
- moved SW3 3.57 mm to (137.2, 82.0)
Connections:
- SW2 pad 1: push button -> push button 1
- SW3 pad 1: push button 1 -> push button
Routing:
- net GND: track 253.6 -> 0.00 mm, vias 1 -> 0
- net 3.3v: track 183.8 -> 0.00 mm
- net SDA: track 130.9 -> 0.00 mm, vias 2 -> 0
- net SCL: track 126.1 -> 0.00 mm
- net BO1: track 80.1 -> 0.00 mm
- net XSHUT 3: track 79.8 -> 0.00 mm
- net 7.4v: track 77.0 -> 0.00 mm
- net 5v: track 65.8 -> 0.00 mm
- net STBY: track 60.9 -> 0.00 mm
- net encoder A1: track 52.7 -> 0.00 mm, vias 1 -> 0
- net BO2: track 37.4 -> 0.00 mm, vias 1 -> 0
- net XSHUT 2: track 36.3 -> 0.00 mm
- net push button 1: track 30.5 -> 0.00 mm
- net XSHUT 1: track 25.7 -> 0.00 mm
- net encoder B2: track 25.3 -> 0.00 mm
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Other:
- outline, holes or cut-outs redrawn
- board text added: "B12"
- board text removed: "STBY"

Commit message: pcb changes
Parts:
- added U9: oled i2c, oled:oled, F.Cu at (162.8, 73.4)
- SW3: value SW_Push -> SW_SPDT_312; footprint push button:push_button -> slide switch:SLIDE SW
- SW4: value SW_SPDT_312 -> SW_Push; footprint slide switch:SLIDE SW -> push button:push_button
- moved SW4 51.7 mm to (137.2, 73.4), turned to 90 degrees
- moved SW3 12.1 mm to (129.5, 72.6), turned to 90 degrees
- moved SW2 9.66 mm to (185.4, 73.4)
- moved U1 8.86 mm to (190.5, 135.1), turned to -90 degrees
- moved U8 7.87 mm to (152.0, 56.9)
- moved U6 4.32 mm to (121.4, 82.5)
- moved U7 4.32 mm to (200.4, 64.8)
Connections:
- SW3 pad 1: push button -> slide_SW
- SW3 pad 2: GND -> 3.3v
- SW3 pad 3: (no net) -> GND
- SW4 pad 1: slide_SW -> push button
- SW4 pad 2: 3.3v -> GND
- SW4 pad 3: GND -> (no net)
Other:
- board size 100 x 100 mm -> 100 x 108 mm

Commit message: pcb changes
Parts:
- moved U5 94.7 mm to (132.3, 46.0), turned to 90 degrees
- moved U2 83.1 mm to (184.9, 61.5), turned to 180 degrees
- moved SW3 69.4 mm to (111.8, 139.7)
- moved SW4 64.3 mm to (195.8, 47.0)
- moved U1 60.5 mm to (130.0, 137.7), turned to 90 degrees
- moved U9 60.2 mm to (161.0, 133.6)
- moved ACC1 31.8 mm to (170.3, 55.2)
- moved U4 29.5 mm to (128.3, 128.3), turned to 90 degrees
- moved U3 29.0 mm to (177.8, 127.8), turned to 90 degrees
- moved SW2 26.9 mm to (180.6, 47.0)
- moved U8 21.7 mm to (150.1, 35.3)
- moved U7 8.18 mm to (196.8, 57.4)
- moved U6 7.37 mm to (121.7, 75.2)
- moved J1 7.19 mm to (206.5, 138.2), turned to 0 degrees
Other:
- board size 100 x 108 mm -> 348.2 x 129.5 mm

Commit message: pcb changes
Parts:
- moved U2 55.6 mm to (132.8, 81.0), turned to 0 degrees
- moved U6 7.33 mm to (114.6, 77.0)
- moved U7 7.33 mm to (204.0, 59.2)
- moved U8 5.85 mm to (150.4, 29.5)
- moved SW3 4.01 mm to (111.8, 135.7), turned to 180 degrees
- moved SW2 3.64 mm to (179.8, 50.5)
- moved SW4 3.64 mm to (195.1, 50.5)
- moved U1 2.79 mm to (130.0, 134.9)
- moved U4 2.79 mm to (128.3, 125.5)
- moved U9 2.79 mm to (161.0, 130.8)
- moved J1 2.79 mm to (206.5, 135.4)
- moved U3 2.29 mm to (177.8, 125.5)
- moved U5 2.29 mm to (134.6, 46.0), turned to -90 degrees
- moved ACC1 0.13 mm to (170.3, 55.4)
Connections:
- U2 pad 26: PWM A -> unconnected-(U2-A0-Pad26)
- U2 pad 27: PWM B -> PWM A
- U2 pad 32: unconnected-(U2-A6-Pad32) -> PWM B
- U5 pad 1: 7.4v -> 7.4vb
Other:
- board size 348.2 x 129.5 mm -> 115.3 x 129.5 mm

Commit message: ll
Routing:
- net GND: track 0.00 -> 365.8 mm
- net 3.3v: track 0.00 -> 313.6 mm, vias 0 -> 1
- net 5v: track 0.00 -> 110.4 mm
