File: micromouse.kicad_pcb (KiCad board)
At the start: 2 copper layers, 115.3 x 129.5 mm, 14 parts, among them J1 XT60-M, SW2 SW_Push, SW3 SW_SPDT_312, SW4 SW_Push, U1 BUCK, U2 STM32 Blackpill, U3 N20 encoder right, U4 N20 encoder left, U5 TB6612FNG, U6 VL53L0X left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

Commit message: routing
Parts:
- removed ACC1: GY-521, GY-521:GY-521_SMD
Connections:
- U2 pad 9: unconnected-(U2-A12-Pad9) -> slide_SW
Routing:
- net XSHUT 1: track 0.00 -> 104.9 mm, vias 0 -> 2
- net slide_SW: track 0.00 -> 86.9 mm, vias 0 -> 1
- net XSHUT 2: track 0.00 -> 72.1 mm, vias 0 -> 3
- net encoder A2: track 0.00 -> 66.7 mm, vias 0 -> 2
- net encoder B2: track 0.00 -> 65.9 mm, vias 0 -> 2
- net encoder A1: track 0.00 -> 65.2 mm, vias 0 -> 2
- net encoder B1: track 0.00 -> 60.8 mm, vias 0 -> 1
- net push button: track 0.00 -> 59.8 mm, vias 0 -> 2
- net XSHUT 3: track 0.00 -> 39.8 mm
- net PWM B: track 0.00 -> 36.9 mm, vias 0 -> 1
- net push button 1: track 0.00 -> 28.7 mm, vias 0 -> 1
- net BO2: track 94.7 -> 92.8 mm, vias 1 -> 2
- net GND: track 387.8 -> 386.4 mm, vias 0 -> 3
- net SCL: track 205.7 -> 206.1 mm, vias 3 -> 5
- net 3.3v: track 352.7 -> 353.1 mm, vias 0 -> 3
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Other:
- board text added: "+"
- board text added: "+ve"
- board text added: "0.96 Inch I2C/IIC 4pin OLED Display"
- board text added: "7.4v"
- board text added: "A01"
- board text added: "AIN1"
- board text added: "AIN2"
- board text added: "AO2"
- board text added: "B01"
- board text added: "BIN1"
- board text added: "BIN2"
- board text added: "BO2"
- board text added: "BlackPill STM32F411CEU6 F411"
- board text added: "C1"
- board text added: "C2"
- board text added: "DC-DC 5V 3A BEC Power Supply Buck Step Down Module"
- board text added: "GA12-N20-6v 500 RPM"
- board text added: "GPIO1"
- board text added: "GY-53 VL53L0X"
- board text added: "HW-290/GY-87 10DOF MPU6050+HMC5883L+BMP180 3-axis Gyro + 3-axis Acceleration + 3-axis Magnetic Field + Air Pressure Sensor"
- board text added: "M1"
- board text added: "M2"
- board text added: "MCU"
- board text added: "PWMA"
- board text added: "PWMB"
- board text added: "SCL"
- board text added: "SDA"
- board text added: "STBY"
- board text added: "Slide Switch SS-12D00 1P2T"
- board text added: "TB6612FNG"
- board text added: "Tactile Push Button"
- board text added: "Vcc"
- board text added: "Vm"
- board text added: "XSHUT"
- board text added: "XT-60"

Commit message: pcb changes
Parts:
- added ACC1: GY-521, GY-521:GY-521_SMD, F.Cu at (170.2, 55.6)
Connections:
- U2 pad 9: slide_SW -> unconnected-(U2-A12-Pad9)

Commit message: final routing
Connections:
- U2 pad 9: unconnected-(U2-A12-Pad9) -> slide_SW
Routing:
- net 3.3v: track 353.1 -> 371.6 mm, vias 3 -> 4
- net GND: track 386.4 -> 390.2 mm
- net SCL: track 206.1 -> 205.4 mm, vias 5 -> 4
- net SDA: track 204.0 -> 203.9 mm, vias 5 -> 4
Other:
- board text added: "HW-290/GY-87 10DOF MPU6050"
- board text removed: "HW-290/GY-87 10DOF MPU6050+HMC5883L+BMP180 3-axis Gyro + 3-axis Acceleration + 3-axis Magnetic Field + Air Pressure Sensor"
Changed lines of the file:
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@@
 	(net 52 "unconnected-(ACC1-INT-Pad8)")
 	(net 53 "unconnected-(ACC1-XDA-Pad5)")
-	(net 54 "unconnected-(U2-A12-Pad9)")
 	(footprint "slide switch:SLIDE SW"
 		(layer "F.Cu")
@@
 		(at 170.18 55.626 90)
 		(property "Reference" "ACC1"
-			(at 8.128 -17.018 90)
+			(at 13.335 -14.986 90)
 			(layer "F.SilkS")
 			(effects
@@
 		(at 130.048 134.874 90)
 		(property "Reference" "U1"
-			(at -1.016 3.508 -90)
+			(at 1.524 4.191 -90)
 			(unlocked yes)
 			(layer "F.SilkS")
@@
 		)
 		(property "Value" "BUCK"
-			(at -1.016 2.008 -90)
+			(at 1.397 1.905 -90)
 			(unlocked yes)
 			(layer "F.Fab")
@@
 			(layers "*.Cu" "*.Mask")
 			(remove_unused_layers no)
-			(net 54 "unconnected-(U2-A12-Pad9)")
+			(net 49 "slide_SW")
 			(pinfunction "A12")
-			(pintype "bidirectional+no_connect")
+			(pintype "bidirectional")
 		)
 		(pad "10" thru_hole circle
@@
 	)
 	(gr_text "GY-53 VL53L0X"
-		(at 109.22 69.469 90)
+		(at 110.744 70.485 90)
 		(layer "F.SilkS")
 		(effects
@@
 	)
 	(gr_text "TB6612FNG"
-		(at 132.461 46.863 0)
+		(at 132.461 51.181 0)
 		(layer "F.SilkS")
 		(effects
@@
 	)
 	(gr_text "BlackPill STM32F411CEU6 F411"
-		(at 155.448 70.739 0)
+		(at 155.575 66.929 0)
 		(layer "F.SilkS")
 		(effects
@@
 	)
 	(gr_text "DC-DC 5V 3A BEC Power Supply \nBuck Step Down Module"
-		(at 127.508 137.033 0)
+		(at 127.635 139.446 0)
 		(layer "F.SilkS")
 		(effects
@@
 		)
 	)
-	(gr_text "HW-290/GY-87 10DOF MPU6050+HMC5883L+BMP180 \n3-axis Gyro + 3-axis Acceleration + 3-axis Magnetic Field \n+ Air Pressure Sensor"
-		(at 147.828 139.446 0)
+	(gr_text "HW-290/GY-87 10DOF MPU6050\n"
+		(at 153.924 50.165 0)
 		(layer "F.SilkS")
 		(effects
@@
 	)
 	(segment
+		(start 153.289 50.927)
+		(end 156.464 50.927)
+		(width 0.5)
+		(layer "F.Cu")
+		(net 1)
+	)
+	(segment
 		(start 174.752 69.0372)
 		(end 174.752 62.243173)
@@
 	)
 	(segment
+		(start 150.368 53.848)
+		(end 153.289 50.927)
+		(width 0.5)
+		(layer "F.Cu")
+		(net 1)
+	)
+	(segment
 		(start 160.782 119.126)
 		(end 162.012 117.896)
@@
 	)
 	(via
+		(at 156.464 50.927)
+		(size 0.7)
+		(drill 0.3)
+		(layers "F.Cu" "B.Cu")
+		(net 1)
+	)
+	(via
 		(at 167.64 51.054)
 		(size 0.7)
@@
 	)
 	(segment
+		(start 167.513 50.927)
+		(end 167.64 51.054)
+		(width 0.5)
+		(layer "B.Cu")
+		(net 1)
+	)
+	(segment
 		(start 138.43 125.476)
 		(end 123.8892 140.0168)
@@
 	)
 	(segment
+		(start 156.464 50.927)
+		(end 167.513 50.927)
+		(width 0.5)
+		(layer "B.Cu")
+		(net 1)
+	)
+	(segment
 		(start 160.782 124.206)
 		(end 143.581 141.407)
@@
 	)
 	(segment
+		(start 152.908 53.848)
+		(end 150.368 56.388)
+		(width 0.5)
+		(layer "B.Cu")
+		(net 2)
+	)
+	(segment
 		(start 154.236 25.712)
 		(end 155.448 26.924)
@@
 	)
 	(segment
+		(start 150.368 56.388)
+		(end 150.241 56.388)
+		(width 0.5)
+		(layer "B.Cu")
+		(net 2)
+	)
+	(segment
 		(start 139.134 61.4752)
 		(end 145.1538 61.4752)
@@
 	)
 	(segment
+		(start 156.083 48.387)
+		(end 156.083 31.623)
+		(width 0.3)
+		(layer "F.Cu")
+		(net 3)
+	)
+	(segment
 		(start 196.596 72.136)
 		(end 189.23 79.502)
@@
 	)
 	(segment
-		(start 158.115 29.591)
-		(end 158.115 47.498)
+		(start 155.702 93.1672)
+		(end 170.942 77.9272)
 		(width 0.3)
 		(layer "F.Cu")
@@
 	)
 	(segment
-		(start 158.115 47.498)
-		(end 158.115 53.594)
+		(start 160.528 27.178)
+		(end 160.528 26.924)
 		(width 0.3)
 		(layer "F.Cu")
@@
 	)
 	(segment
-		(start 155.702 93.1672)
-		(end 170.942 77.9272)
+		(start 156.083 48.387)
+		(end 157.988 50.292)
 		(width 0.3)
 		(layer "F.Cu")
@@
 	)
 	(segment
-		(start 160.528 27.178)
-		(end 158.115 29.591)
+		(start 156.083 31.623)
+		(end 160.528 27.178)
 		(width 0.3)
 		(layer "F.Cu")
@@
 	)
 	(segment
-		(start 141.986 44.958)
-		(end 130.048 44.958)
+		(start 157.988 50.292)
+		(end 157.988 53.848)
 		(width 0.3)
 		(layer "F.Cu")
@@
 	)
 	(segment
-		(start 160.528 26.924)
-		(end 160.528 27.178)
+		(start 141.986 44.958)
+		(end 130.048 44.958)
 		(width 0.3)
 		(layer "F.Cu")
@@
 	)
 	(via
-		(at 158.115 53.594)
-		(size 0.7)
-		(drill 0.3)
-		(layers "F.Cu" "B.Cu")
-		(net 3)
-	)
-	(via
-		(at 158.115 48.26)
+		(at 156.083 48.387)
 		(size 0.7)
 		(drill 0.3)
@@
 	)
 	(segment
+		(start 158.115 53.975)
+		(end 158.496 53.975)
+		(width 0.3)
+		(layer "B.Cu")
+		(net 3)
+	)
+	(segment
+		(start 157.988 53.848)
+		(end 158.115 53.975)
+		(width 0.3)
+		(layer "B.Cu")
+		(net 3)
+	)
+	(segment
 		(start 113.126 61.88)
 		(end 113.126 65.69)
@@
 	)
 	(segment
-		(start 157.353 47.498)
-		(end 144.526 47.498)
+		(start 155.194 47.498)
+		(end 156.083 48.387)
 		(width 0.3)
 		(layer "B.Cu")
@@
 	)
 	(segment
-		(start 172.5168 79.502)
-		(end 189.23 79.502)
+		(start 158.496 53.975)
+		(end 164.434 59.913)
 		(width 0.3)
 		(layer "B.Cu")
@@
 	)
 	(segment
-		(start 170.942 77.9272)
-		(end 172.5168 79.502)
+		(start 172.5168 79.502)
+		(end 189.23 79.502)
 		(width 0.3)
 		(layer "B.Cu")
@@
 	)
 	(segment
-		(start 158.115 53.594)
-		(end 164.434 59.913)
+		(start 170.942 77.9272)
+		(end 172.5168 79.502)
 		(width 0.3)
 		(layer "B.Cu")
@@
 	)
 	(segment
-		(start 158.115 48.26)
-		(end 157.353 47.498)
+		(start 144.526 47.498)
+		(end 141.986 44.958)
 		(width 0.3)
 		(layer "B.Cu")
@@
 	(segment
 		(start 144.526 47.498)
-		(end 141.986 44.958)
+		(end 155.194 47.498)
 		(width 0.3)
 		(layer "B.Cu")
@@
 	)
 	(segment
+		(start 155.575 34.925)
+		(end 155.575 29.591)
+		(width 0.3)
+		(layer "F.Cu")
+		(net 4)
+	)
+	(segment
 		(start 157.988 26.924)
 		(end 157.988 27.178)
@@
 	)
 	(segment
-		(start 155.575 29.591)
-		(end 155.575 53.594)
+		(start 157.988 27.178)
+		(end 155.575 29.591)
 		(width 0.3)
 		(layer "F.Cu")
@@
 	)
 	(segment
-		(start 157.988 27.178)
-		(end 155.575 29.591)
+		(start 142.748 47.752)
+		(end 155.575 34.925)
 		(width 0.3)
 		(layer "F.Cu")
@@
 	)
 	(via
-		(at 155.5115 53.5305)
-		(size 0.7)
-		(drill 0.3)
-		(layers "F.Cu" "B.Cu")
-		(net 4)
-	)
-	(via
 		(at 190.754 75.946)
 		(size 0.7)
@@
 	)
 	(segment
-		(start 154.051 52.07)
-		(end 155.5115 53.5305)
+		(start 159.67 69.1952)
+		(end 168.402 77.9272)
 		(width 0.3)
 		(layer "B.Cu")
@@
 	)
 	(segment
-		(start 124.618 52.928)
-		(end 129.794 47.752)
+		(start 147.066 52.07)
+		(end 153.67 52.07)
 		(width 0.3)
 		(layer "B.Cu")
@@
 	)
 	(segment
-		(start 155.575 53.594)
-		(end 159.67 57.689)
+		(start 124.618 52.928)
+		(end 129.794 47.752)
 		(width 0.3)
 		(layer "B.Cu")
@@
 	)
 	(segment
-		(start 147.066 52.07)
-		(end 154.051 52.07)
-		(width 0.3)
-		(layer "B.Cu")
-		(net 4)
-	)
-	(segment
-		(start 159.67 57.689)
+		(start 159.67 58.07)
 		(end 159.67 69.1952)
 		(width 0.3)
@@
 	)
 	(segment
+		(start 155.448 53.848)
+		(end 159.67 58.07)
+		(width 0.3)
+		(layer "B.Cu")
+		(net 4)
+	)
+	(segment
+		(start 153.67 52.07)
+		(end 155.448 53.848)
+		(width 0.3)
+		(layer "B.Cu")
+		(net 4)
+	)
+	(segment
 		(start 173.5328 83.058)
 		(end 187.452 83.058)
@@
 		(width 0.3)
 		(layer "B.Cu")
-		(net 4)
-	)
-	(segment
-		(start 159.67 69.1952)
-		(end 168.402 77.9272)
-		(width 0.3)
-		(layer "B.Cu")
