File: _autosave-micromouse.kicad_pcb (KiCad board)
At the start: 2 copper layers, 115.3 x 122.3 mm, 14 parts, among them J1 XT60-M, SW2 SW_Push, SW3 SW_SPDT_312, SW4 SW_Push, U1 BUCK, U2 STM32 Blackpill, U3 N20 encoder right, U4 N20 encoder left, U5 TB6612FNG, U6 VL53L0X left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

Commit message: pcb
Parts:
- SW2, SW4: footprint push button:push_button -> push button 1:SW_VS-1213-67-160GF
- moved U7 2.27 mm to (183.3, 50.1)
- moved SW4 1.72 mm to (129.1, 63.4)
- moved SW2 1.69 mm to (170.9, 63.3)
- moved U6 1.08 mm to (116.8, 67.8)
Routing:
- net XSHUT 3: track 51.2 -> 53.9 mm
- net SCL: track 216.0 -> 218.2 mm
- net XSHUT 1: track 50.6 -> 51.9 mm
- net 3.3v: track 268.7 -> 267.7 mm
- net SDA: track 194.5 -> 193.7 mm
Other:
- outline, holes or cut-outs redrawn

Commit message: pcb
Parts:
- added G***: LOGO, rnc:rnc3, F.Cu at (129.7, 49.1)
- added SW1: SW_SPST, power switch:battery_sw, F.Cu at (195.4, 131.8)
Connections:
- U5 pad 2: 5v -> 3.3v
Routing:
- net 3.3v: track 267.7 -> 324.4 mm
- net 7.4vb: track 11.5 -> 38.3 mm
- net 5v: track 104.5 -> 83.3 mm
- net 7.4v: track 0.00 -> 15.0 mm
- net AIN1: track 45.7 -> 47.5 mm
- net XSHUT 1: track 51.9 -> 50.2 mm
- net XSHUT 3: track 53.9 -> 52.2 mm
- net BO2: track 30.1 -> 31.1 mm
- net AIN2: track 45.7 -> 46.5 mm
Other:
- board size 115.3 x 122.3 mm -> 115 x 122.4 mm
